File: hardware/sc.brd (EAGLE design)
At the start: 82.8 x 56 mm, 99 parts, among them IC1 PB137ACV, IC2 INA168, Q1 si2305cd, Q2 8MHz 18pF, Q3 IRFR5305, T1 BC846, U1 SPX5205 3v3, U6 microSD Socket, X3 MKDSN1,5/4-5,08, Y1 32768Hz CFPX-217 12.5pF

Commit message: lower LED power
Parts:
- R12, R17, R20, R27: value 1K -> 2k2
Changed lines of the file:
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@@
 <element name="R5" library="rcl" package="R0805W" value="4.7k" x="77.3" y="45.6"/>
 <element name="LED2" library="led" package="CHIP-LED0805" value="orange" x="54.5" y="28.3" rot="R180"/>
-<element name="R27" library="rcl" package="R0805W" value="1K" x="54.5" y="23.3" rot="R90"/>
+<element name="R27" library="rcl" package="R0805W" value="2k2" x="54.5" y="23.3" rot="R90"/>
 <element name="U$2" library="Simplex-Fuses" package="1210" value="RESETTABLE" x="24.1" y="14.3" rot="R270"/>
 <element name="IC1" library="linear" package="TO220V" value="PB137ACV" x="0.5" y="41.9" rot="R90"/>
@@
 <element name="C27" library="SparkFun-Capacitors" package="PANASONIC_D" value="10uF" x="11.8" y="51" rot="R270"/>
 <element name="C26" library="SparkFun-Capacitors" package="PANASONIC_D" value="1uF" x="11.8" y="40.3" rot="R90"/>
-<element name="R12" library="rcl" package="R0805W" value="1K" x="34.2" y="30.2"/>
+<element name="R12" library="rcl" package="R0805W" value="2k2" x="34.2" y="30.2"/>
 <element name="LED3" library="led" package="CHIP-LED0805" value="green" x="34.2" y="32.4" rot="R270"/>
-<element name="R17" library="rcl" package="R0805W" value="1K" x="34.2" y="25.8"/>
+<element name="R17" library="rcl" package="R0805W" value="2k2" x="34.2" y="25.8"/>
 <element name="LED4" library="led" package="CHIP-LED0805" value="green" x="34.2" y="28" rot="R270"/>
-<element name="R20" library="rcl" package="R0805W" value="1K" x="34.2" y="21.4"/>
+<element name="R20" library="rcl" package="R0805W" value="2k2" x="34.2" y="21.4"/>
 <element name="LED5" library="led" package="CHIP-LED0805" value="green" x="34.2" y="23.6" rot="R270"/>
 <element name="R21" library="rcl" package="R0805W" value="220k" x="34.2" y="43.4" rot="R180"/>

Commit message: keep track of programming time
Parts:
- R21, R28, R36: value 220k -> 1M
Changed lines of the file:
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@@
 <element name="R20" library="rcl" package="R0805W" value="2k2" x="34.2" y="21.4"/>
 <element name="LED5" library="led" package="CHIP-LED0805" value="green" x="34.2" y="23.6" rot="R270"/>
-<element name="R21" library="rcl" package="R0805W" value="220k" x="34.2" y="43.4" rot="R180"/>
+<element name="R21" library="rcl" package="R0805W" value="1M" x="34.2" y="43.4" rot="R180"/>
 <element name="LED6" library="led" package="CHIP-LED0805" value="green" x="34.2" y="45.6" rot="R90"/>
-<element name="R28" library="rcl" package="R0805W" value="220k" x="34.2" y="34.6" rot="R180"/>
+<element name="R28" library="rcl" package="R0805W" value="1M" x="34.2" y="34.6" rot="R180"/>
 <element name="LED7" library="led" package="CHIP-LED0805" value="green" x="34.2" y="36.8" rot="R90"/>
-<element name="R36" library="rcl" package="R0805W" value="220k" x="34.2" y="39" rot="R180"/>
+<element name="R36" library="rcl" package="R0805W" value="1M" x="34.2" y="39" rot="R180"/>
 <element name="LED8" library="led" package="CHIP-LED0805" value="green" x="34.2" y="41.2" rot="R90"/>
 <element name="D2" library="diode" package="C1702-05" value="SB560" x="14.1" y="32.7" rot="R180"/>
