File: hardware/sc.brd (EAGLE design)
At the start: 65 x 56 mm, 88 parts, among them IC1 PB137ACV, IC2 LM2675M-ADJ, Q1 si2305cd, Q2 IRFR5305, Q3 IRFR5305, T1 BC846, T2 BC846, T3 BC846, U1 SPX5205 3v3, X1 prog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

Commit message: rev4
Parts:
- moved U$7 2.04 mm to (61.1, 8.63)
Other:
- board text added: "sc rev04 Petre Rodan 201511"
- board text removed: "Petre Rodan 201511 rev1"
Changed lines of the file:
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@@
 <?xml version="1.0" encoding="utf-8"?>
 <!DOCTYPE eagle SYSTEM "eagle.dtd">
-<eagle version="7.3.0">
+<eagle version="7.5.0">
 <drawing>
 <settings>
@@
 <vertex x="35.4" y="44.9"/>
 </polygon>
-<text x="39.1" y="6.2" size="0.8128" layer="108" ratio="15">Petre Rodan 201511 rev1</text>
+<text x="39.1" y="6.2" size="0.8128" layer="108" ratio="15">sc rev04  Petre Rodan 201511</text>
 <text x="39.1" y="4.6" size="0.8128" layer="108" ratio="15">github.com/rodan/solar-charger</text>
 <text x="45.3" y="48.3" size="0.8128" layer="108" ratio="15">ts</text>
@@
 <element name="U$1" library="TI_MSP430_v16" package="PT48" value="F55[0/1]X---PT48" x="50.8" y="18"/>
 <element name="U$17" library="Simplex-ICs" package="S-PVQFN-N16" value="BQ24072" x="38.1" y="45.9" rot="R270"/>
-<element name="U$7" library="SparkFun" package="OSHW-LOGO-M" value="OSHW-LOGOM" x="59.09" y="8.23"/>
+<element name="U$7" library="SparkFun" package="OSHW-LOGO-M" value="OSHW-LOGOM" x="61.09" y="8.63"/>
 <element name="U1" library="SparkFun" package="SOT23-5" value="SPX5205 3v3" x="45.2" y="35.7" rot="R270"/>
 <element name="X3" library="con-phoenix-508" package="MKDSN1,5/4-5,08" value="MKDSN1,5/4-5,08" x="10.23" y="4.25" rot="R180">
