File: hardware/sc.sch (EAGLE design)
At the start: 88 parts, among them IC1 PB137ACV, IC2 LM2675M-ADJ, Q1 si2305cd, Q2 IRFR5305, Q3 IRFR5305, T1 BC846, T2 BC846, T3 BC846, U1 SPX5205 3v3, X1 prog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

Commit message: rev4
Other:
- note added: "04"
- note removed: "02"
Changed lines of the file:
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@@
 <?xml version="1.0" encoding="utf-8"?>
 <!DOCTYPE eagle SYSTEM "eagle.dtd">
-<eagle version="7.3.0">
+<eagle version="7.5.0">
 <drawing>
 <settings>
@@
 <sheet>
 <plain>
-<text x="416.56" y="10.16" size="3.81" layer="97">02</text>
+<text x="416.56" y="10.16" size="3.81" layer="97">04</text>
 <text x="241.3" y="177.8" size="1.778" layer="97">uC pins: 7 11 28</text>
 <text x="322.58" y="304.8" size="1.778" layer="97">ILIM=1610/R15</text>
