File: rev2/hardware/sc.sch (EAGLE design)
At the start: 81 parts, among them IC1 PB137ACV, IC2 LM2675M-ADJ, Q1 si2305cd, Q2 IRFR5305, Q3 IRFR5305, T1 BC846, U1 SPX5205 3v3, X3 MKDSN1,5/4-5,08, X4 ts, X5 i2c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

Commit message: rev2 routing 2/3
Parts:
- removed R40: 0R, rcl:R-EU_R0805W
- removed X7: prog, Simplex-Connectors:MOLEX_6VERTICAL
- added R10, R12, R13: 0R_0805, Simplex-Jumpers:0R_0805
- added X1: prog, Simplex-Connectors:MOLEX_6HORIZONTAL
Connections:
- net +3V3: now also X1.4; no longer X7.3
- net BAT_DIV: now also U$1.2; no longer U$1.3
- net CE: now also U$1.1
- net GND: now also LED6.C, LED7.C, LED8.C, R10.P$2, R12.P$2, R13.P$1, R13.P$2, X1.1; no longer R40.2, X7.6
- net PV_DIV: now also U$1.4; no longer U$1.2
- net PV_EN: now also U$1.15; no longer U$1.22
- net RST: now also X1.2; no longer X7.5
- net RX: now also X1.5; no longer X7.2
- net STATUS: now also U$1.16; no longer U$1.36
- net TEST: now also X1.3; no longer X7.4
- net THERM: now also U$1.6; no longer U$1.5
- net TH_EN: now also U$1.5; no longer U$1.21
- net TX: now also X1.6; no longer X7.1
- net VBAT_DIV: now also U$1.3; no longer U$1.1
- net VBAT_GND: now also R10.P$1, R12.P$1; no longer LED6.C, LED7.C, LED8.C, R40.1

Commit message: board ready
Parts:
- added C14: 100nF, rcl:C-EUC0805
- added R29: 470, rcl:R-EU_R0805W
- added R32: 100k, rcl:R-EU_R0805W
- added T2, T3: BC846, transistor:BC846
- C11: value 1uF -> 10nF
- R19: value 10k -> 220k
- R3: value 100k -> 220k
- R30: value 1M -> 220k
- R31: value 10k -> 1M
- SJ1: value JUMPER-PAD-3-2OF3_NC_BY_PASTE -> sel_in
- SJ2: value JUMPER-PAD-2-NC_BY_PASTE -> i2c_pwr
Connections:
- new net N$20: R29.2, U$1.1
- new net N$22: C14.1, R31.1, T2.B, T3.C
- new net N$23: R32.1, T3.B
- net CE: now also R29.1, R32.2; no longer R31.1, U$1.1
- net GND: now also C14.2, T2.E, T3.E; no longer C11.1, R30.1
- net N$16: now also R30.1, T2.C; no longer R30.2, R31.2
- net N$49: now also C11.1
- net VBAT: now also R30.2, R31.2
Other:
- note added: "02"
- note removed: "03"
- moved on the sheet: C11, C26, C27, D2, IC1, Q2, Q3, R16, R19, R2, R30, R31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
