File: hardware/rev4/sc.brd (EAGLE design)
At the start: 65 x 56 mm, 88 parts, among them IC1 PB137ACV, IC2 LM2675M-ADJ, Q1 si2305cd, Q2 IRFR5305, Q3 IRFR5305, T1 BC846, T2 BC846, T3 BC846, U1 SPX5205 3v3, X1 prog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

Commit message: control pins working
Parts:
- C16, C26: value 1uF -> 1uF DNP
- C25: value 100nF -> 100nF DNP
- C27: value 10uF -> 10uF DNP
- IC1: value PB137ACV -> PB137ACV DNP
- Q1: value si2305cd -> si2305cd DNP
- R11: value 30k -> 30k DNP
- R3: value 220k -> 220k DNP
- R6, R7: value 4.7k -> 470
- R8: value 10k -> 10k DNP
Changed lines of the file:
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@@
 <element name="C10" library="rcl" package="C0805" value="470nF" x="45.2" y="10.1" rot="R180"/>
 <element name="C12" library="rcl" package="PANASONIC_D" value="100uF, 16V" x="27.97" y="50.19" rot="R180"/>
-<element name="C16" library="rcl" package="C0805" value="1uF" x="25.1" y="24.3" rot="R180"/>
+<element name="C16" library="rcl" package="C0805" value="1uF DNP" x="25.1" y="24.3" rot="R180"/>
 <element name="C17" library="rcl" package="C0805" value="100nF" x="38.7" y="19.1"/>
 <element name="C18" library="rcl" package="C0805" value="100nF" x="36" y="23.8" rot="R270"/>
@@
 <element name="C23" library="rcl" package="C0805" value="22pF" x="38.7" y="16.5" rot="R180"/>
 <element name="C24" library="rcl" package="C0805" value="22pF" x="38.7" y="14.4" rot="R180"/>
-<element name="C25" library="rcl" package="C0805" value="100nF" x="25.1" y="12.7"/>
-<element name="C26" library="SparkFun-Capacitors" package="PANASONIC_D" value="1uF" x="13.16" y="21.39" rot="R180"/>
-<element name="C27" library="SparkFun-Capacitors" package="PANASONIC_D" value="10uF" x="17.68" y="14.2" rot="R180"/>
+<element name="C25" library="rcl" package="C0805" value="100nF DNP" x="25.1" y="12.7"/>
+<element name="C26" library="SparkFun-Capacitors" package="PANASONIC_D" value="1uF DNP" x="13.16" y="21.39" rot="R180"/>
+<element name="C27" library="SparkFun-Capacitors" package="PANASONIC_D" value="10uF DNP" x="17.68" y="14.2" rot="R180"/>
 <element name="C3" library="rcl" package="C1206" value="10uF" x="45.2" y="40.7"/>
 <element name="C38" library="rcl" package="C1206" value="4u7" x="38.62" y="50.7" rot="R180"/>
@@
 </element>
 <element name="D2" library="diode" package="C1702-05" value="SB560" x="6.98" y="21.65" rot="R270"/>
-<element name="IC1" library="linear" package="TO220V" value="PB137ACV" x="0.34" y="28.73" rot="R90"/>
+<element name="IC1" library="linear" package="TO220V" value="PB137ACV DNP" x="0.34" y="28.73" rot="R90"/>
 <element name="IC2" library="Simplex-ICs" package="SO-08" value="LM2675M-ADJ" x="18.58" y="45.92" rot="R180"/>
 <element name="JP2" library="SparkFun-Connectors" package="1X02" value="thermistor" x="2.79" y="18.98" rot="R90"/>
@@
 <element name="LED7" library="led" package="CHIP-LED0805" value="green" x="30.5" y="8.5" rot="R270"/>
 <element name="LED8" library="led" package="CHIP-LED0805" value="green" x="30.5" y="12.7" rot="R270"/>
-<element name="Q1" library="Simplex-DiscreteSemi" package="SOT23-3_POWER@1" value="si2305cd" x="25" y="21.7" rot="R90"/>
+<element name="Q1" library="Simplex-DiscreteSemi" package="SOT23-3_POWER@1" value="si2305cd DNP" x="25" y="21.7" rot="R90"/>
 <element name="Q2" library="transistor-power" package="D-PAK_TO252AA" value="IRFR5305" x="13.15" y="32.22" rot="R270"/>
 <element name="Q3" library="transistor-power" package="D-PAK_TO252AA" value="IRFR5305" x="6.95" y="14.25" rot="R270"/>
 <element name="R1" library="rcl" package="R0805W" value="1.5K 1%" x="17.68" y="51.5"/>
-<element name="R11" library="rcl" package="R0805W" value="30k" x="25.1" y="14.8" rot="R180"/>
+<element name="R11" library="rcl" package="R0805W" value="30k DNP" x="25.1" y="14.8" rot="R180"/>
 <element name="R14" library="rcl" package="R0805W" value="47k" x="61.6" y="31.9" rot="R270"/>
 <element name="R15" library="rcl" package="R0805W" value="47k" x="59.5" y="31.9" rot="R270"/>
@@
 <element name="R27" library="rcl" package="R0805W" value="4.7k" x="51" y="32.9"/>
 <element name="R28" library="rcl" package="R0805W" value="1M" x="30.5" y="10.6"/>
-<element name="R3" library="rcl" package="R0805W" value="220k" x="25.1" y="19"/>
+<element name="R3" library="rcl" package="R0805W" value="220k DNP" x="25.1" y="19"/>
 <element name="R36" library="rcl" package="R0805W" value="1M" x="30.5" y="14.8"/>
 <element name="R37" library="rcl" package="R0805W" value="100k" x="30.5" y="6.4"/>
-<element name="R6" library="rcl" package="R0805W" value="4.7k" x="57.4" y="31.9" rot="R270"/>
-<element name="R7" library="rcl" package="R0805W" value="4.7k" x="55.3" y="31.9" rot="R270"/>
-<element name="R8" library="rcl" package="R0805W" value="10k" x="25.1" y="16.9" rot="R180"/>
+<element name="R6" library="rcl" package="R0805W" value="470" x="57.4" y="31.9" rot="R270"/>
+<element name="R7" library="rcl" package="R0805W" value="470" x="55.3" y="31.9" rot="R270"/>
+<element name="R8" library="rcl" package="R0805W" value="10k DNP" x="25.1" y="16.9" rot="R180"/>
 <element name="R9" library="rcl" package="R0805W" value="4.75k 1%" x="21.8" y="51.5"/>
 <element name="T1" library="transistor" package="SOT23" value="BC846" x="25.1" y="7.5" rot="R90"/>

Commit message: adc, rtc work
Parts:
- R22: value 2M -> 1M2
- R24: value 220k -> 100k
- R32: value 100k -> DNP 100k
- R4: value 2M -> 680K
- R5: value 1M3 -> 330k
- R9: value 4.75k 1% -> 4K3
Changed lines of the file:
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@@
 <element name="R20" library="rcl" package="R0805W" value="1k1" x="41.5" y="38.4" rot="R270"/>
 <element name="R21" library="rcl" package="R0805W" value="1M" x="30.5" y="19"/>
-<element name="R22" library="rcl" package="R0805W" value="2M" x="33.8" y="23.8" rot="R90"/>
+<element name="R22" library="rcl" package="R0805W" value="1M2" x="33.8" y="23.8" rot="R90"/>
 <element name="R23" library="rcl" package="R0805W" value="4.7k" x="51" y="30.8"/>
-<element name="R24" library="rcl" package="R0805W" value="220k" x="38" y="23.8" rot="R270"/>
+<element name="R24" library="rcl" package="R0805W" value="100k" x="38" y="23.8" rot="R270"/>
 <element name="R25" library="rcl" package="R0805W" value="2M" x="33.8" y="27.9" rot="R90"/>
 <element name="R26" library="rcl" package="R0805W" value="330k" x="38" y="27.9" rot="R270"/>
@@
 <element name="R7" library="rcl" package="R0805W" value="470" x="55.3" y="31.9" rot="R270"/>
 <element name="R8" library="rcl" package="R0805W" value="10k DNP" x="25.1" y="16.9" rot="R180"/>
-<element name="R9" library="rcl" package="R0805W" value="4.75k 1%" x="21.8" y="51.5"/>
+<element name="R9" library="rcl" package="R0805W" value="4K3" x="21.8" y="51.5"/>
 <element name="T1" library="transistor" package="SOT23" value="BC846" x="25.1" y="7.5" rot="R90"/>
 <element name="TP6" library="testpad" package="TP12R" value="TPTP12R" x="34.3" y="5.5">
@@
 <element name="X5" library="Simplex-Connectors" package="0530480401" value="i2c" x="49.7" y="54"/>
 <element name="Y1" library="Simplex-FreqCtrl" package="CRYSTAL-SMD-3.2X1.5" value="32768Hz CFPX-217 12.5pF" x="42.1" y="15.5" rot="R90"/>
-<element name="R4" library="rcl" package="R0805W" value="2M" x="38" y="32" rot="R270"/>
-<element name="R5" library="rcl" package="R0805W" value="1M3" x="33.8" y="32" rot="R90"/>
+<element name="R4" library="rcl" package="R0805W" value="680K" x="38" y="32" rot="R270"/>
+<element name="R5" library="rcl" package="R0805W" value="330k" x="33.8" y="32" rot="R90"/>
 <element name="C13" library="rcl" package="C0805" value="100nF" x="35.9" y="32" rot="R90"/>
 <element name="SJ1" library="SparkFun-Passives" package="PAD-JUMPER-3-2OF3_NC_BY_PASTE_YES_SILK_FULL_BOX" value="sel_in" x="37.9" y="36.7"/>
@@
 <element name="T3" library="transistor" package="SOT23" value="BC846" x="30.5" y="31.1" rot="R180"/>
 <element name="R31" library="rcl" package="R0805W" value="1M" x="25.1" y="28.8" rot="R180"/>
-<element name="R32" library="rcl" package="R0805W" value="100k" x="30.5" y="34.6"/>
+<element name="R32" library="rcl" package="R0805W" value="DNP 100k" x="30.5" y="34.6"/>
 <element name="C14" library="rcl" package="C0805" value="100nF" x="30.5" y="27.3" rot="R180"/>
 </elements>

Commit message: testing stage
Parts:
- R17: value 3k -> 8k9
- R20: value 1k1 -> 8k
Changed lines of the file:
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@@
 <element name="R15" library="rcl" package="R0805W" value="47k" x="59.5" y="31.9" rot="R270"/>
 <element name="R16" library="rcl" package="R0805W" value="100k" x="30.5" y="2.3"/>
-<element name="R17" library="rcl" package="R0805W" value="3k" x="42.4" y="51.6" rot="R90"/>
+<element name="R17" library="rcl" package="R0805W" value="8k9" x="42.4" y="51.6" rot="R90"/>
 <element name="R18" library="rcl" package="R0805W" value="DNP 10k th" x="45.8" y="51"/>
 <element name="R19" library="rcl" package="R0805W" value="220k" x="25.1" y="2.3" rot="R180"/>
 <element name="R2" library="rcl" package="R0805W" value="10k" x="25.1" y="4.4"/>
-<element name="R20" library="rcl" package="R0805W" value="1k1" x="41.5" y="38.4" rot="R270"/>
+<element name="R20" library="rcl" package="R0805W" value="8k" x="41.5" y="38.4" rot="R270"/>
 <element name="R21" library="rcl" package="R0805W" value="1M" x="30.5" y="19"/>
 <element name="R22" library="rcl" package="R0805W" value="1M2" x="33.8" y="23.8" rot="R90"/>

Commit message: add README files
Parts:
- D2: value SB560 -> SB560 DNP
Changed lines of the file:
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@@
 <attribute name="PROD_ID" value="DIO-08053" x="18.17" y="38.97" size="1.778" layer="27" rot="R180" display="off"/>
 </element>
-<element name="D2" library="diode" package="C1702-05" value="SB560" x="6.98" y="21.65" rot="R270"/>
+<element name="D2" library="diode" package="C1702-05" value="SB560 DNP" x="6.98" y="21.65" rot="R270"/>
 <element name="IC1" library="linear" package="TO220V" value="PB137ACV DNP" x="0.34" y="28.73" rot="R90"/>
 <element name="IC2" library="Simplex-ICs" package="SO-08" value="LM2675M-ADJ" x="18.58" y="45.92" rot="R180"/>
